File: meidi.kicad_pcb (KiCad board)
At the start: 2 copper layers, 115.5 x 104.5 mm, 9 parts, among them J1 TOUCH_KEYS, SW1 SW_Push, SW2 SW_Push, SW3 SW_Push, SW4 RotaryEncoder_Switch_MP, U1 Waveshare ESP32-S3-ZERO

Commit message: routed the pcb
Routing:
- net GND: track 0.00 -> 314.3 mm
- net /TOUCH2: track 0.00 -> 225.7 mm
- net /TOUCH1: track 0.00 -> 172.4 mm
- net /SWITCH3: track 0.00 -> 159.2 mm, vias 0 -> 1
- net /SWITCH2: track 0.00 -> 143.6 mm
- net /SWITCH1: track 0.00 -> 115.8 mm
- net +3V3: track 0.00 -> 106.8 mm, vias 0 -> 1
- net /R_POT1: track 0.00 -> 105.4 mm, vias 0 -> 1
- net /ENC1_B: track 0.00 -> 96.8 mm
- net /TOUCH3: track 0.00 -> 87.6 mm, vias 0 -> 2
- net /ENC1_A: track 0.00 -> 87.3 mm
- net /TOUCH4: track 0.00 -> 66.4 mm, vias 0 -> 2
- net /TOUCH5: track 0.00 -> 57.3 mm, vias 0 -> 1
- net /TOUCH7: track 0.00 -> 47.8 mm, vias 0 -> 1
- net /SLIDE2: track 0.00 -> 45.8 mm
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
Commit message: addd readme + produced files
Other:
- board text added: "MUSIC IS MY LOVE LANGUAGE"
